File: KiCAD/BP-Extension.sch (KiCad schematic (older format))
At the start: 7 parts, among them P1 CONN_01X06, SW1 SW_Push, U1 BP, U2 RFM69

Commit message: On the way to rev2
Parts:
- added R2, R3: R, Resistors_SMD:R_0805_HandSoldering, symbol R
- added U3: M24M02-DR, Housings_SOIC:SOIC-8_3.9x4.9mm_Pitch1.27mm, symbol M24M02-DR
Connections:
- net +3V3: now also R2.2, R3.2, U3.8 (Vcc)
- net GND: now also U3.3 (E2), U3.4 (Vss), U3.7 (^WC)
- net SCL: now reaches U1.PB6
- net SCL: now also R3.1, U3.6 (SCL)
- net SDA: now reaches U1.PB7
- net SDA: now also R2.1, U3.5 (SDA)
Changed lines of the file:
@@
 LIBS:switches
 LIBS:mechanical
+LIBS:m24m02-dr
 LIBS:BP-Extension-cache
 EELAYER 25 0
@@
 Wire Wire Line
 	9600 5050 9600 4900
+$Comp
+L M24M02-DR U3
+U 1 1 58A82BD6
+P 3150 6200
+F 0 "U3" H 3350 5750 60  0000 C CNN
+F 1 "M24M02-DR" H 2800 5750 60  0000 C CNN
+F 2 "Housings_SOIC:SOIC-8_3.9x4.9mm_Pitch1.27mm" H 3150 6200 60  0001 C CNN
+F 3 "" H 3150 6200 60  0001 C CNN
+	1    3150 6200
+	1    0    0    -1
+$EndComp
+$Comp
+L GND #PWR011
+U 1 1 58A82D4A
+P 3150 6850
+F 0 "#PWR011" H 3150 6600 50  0001 C CNN
+F 1 "GND" H 3150 6700 50  0000 C CNN
+F 2 "" H 3150 6850 50  0000 C CNN
+F 3 "" H 3150 6850 50  0000 C CNN
+	1    3150 6850
+	1    0    0    -1
+$EndComp
+$Comp
+L +3.3V #PWR012
+U 1 1 58A82DFD
+P 3150 5550
+F 0 "#PWR012" H 3150 5400 50  0001 C CNN
+F 1 "+3.3V" H 3150 5690 50  0000 C CNN
+F 2 "" H 3150 5550 50  0000 C CNN
+F 3 "" H 3150 5550 50  0000 C CNN
+	1    3150 5550
+	1    0    0    -1
+$EndComp
+Wire Wire Line
+	3150 6800 3150 6850
+Wire Wire Line
+	3150 5600 3150 5550
+$Comp
+L GND #PWR013
+U 1 1 58A82FE6
+P 3700 6400
+F 0 "#PWR013" H 3700 6150 50  0001 C CNN
+F 1 "GND" H 3700 6250 50  0000 C CNN
+F 2 "" H 3700 6400 50  0000 C CNN
+F 3 "" H 3700 6400 50  0000 C CNN
+	1    3700 6400
+	1    0    0    -1
+$EndComp
+Wire Wire Line
+	3600 6300 3700 6300
+Wire Wire Line
+	3700 6100 3700 6400
+Wire Wire Line
+	3600 6100 3700 6100
+Connection ~ 3700 6300
+Text GLabel 4900 2700 2    60   Input ~ 0
+SDA
+Text GLabel 4900 2800 2    60   Input ~ 0
+SCL
+Text GLabel 2600 6300 0    60   Input ~ 0
+SDA
+Text GLabel 2600 6100 0    60   Input ~ 0
+SCL
+Wire Wire Line
+	2600 6100 2700 6100
+Wire Wire Line
+	2600 6300 2700 6300
+$Comp
+L R R2
+U 1 1 58A83AC9
+P 4600 2550
+F 0 "R2" V 4680 2550 50  0000 C CNN
+F 1 "R" V 4600 2550 50  0000 C CNN
+F 2 "Resistors_SMD:R_0805_HandSoldering" V 4530 2550 50  0001 C CNN
+F 3 "" H 4600 2550 50  0000 C CNN
+	1    4600 2550
+	-1   0    0    1
+$EndComp
+$Comp
+L R R3
+U 1 1 58A83B54
+P 4800 2650
+F 0 "R3" V 4880 2650 50  0000 C CNN
+F 1 "R" V 4800 2650 50  0000 C CNN
+F 2 "Resistors_SMD:R_0805_HandSoldering" V 4730 2650 50  0001 C CNN
+F 3 "" H 4800 2650 50  0000 C CNN
+	1    4800 2650
+	-1   0    0    1
+$EndComp
+Wire Wire Line
+	4000 2700 4900 2700
+Connection ~ 4600 2700
+Wire Wire Line
+	4000 2800 4900 2800
+Connection ~ 4800 2800
+$Comp
+L +3.3V #PWR014
+U 1 1 58A83D13
+P 4700 2300
+F 0 "#PWR014" H 4700 2150 50  0001 C CNN
+F 1 "+3.3V" H 4700 2440 50  0000 C CNN
+F 2 "" H 4700 2300 50  0000 C CNN
+F 3 "" H 4700 2300 50  0000 C CNN
+	1    4700 2300
+	1    0    0    -1
+$EndComp
+Wire Wire Line
+	4600 2300 4800 2300
+Wire Wire Line
+	4600 2300 4600 2400
+Wire Wire Line
+	4800 2300 4800 2500
+Connection ~ 4700 2300
 $EndSCHEMATC
