File: KiCAD/BPnode-BB.sch (KiCad schematic (older format))
At the start: 10 parts, among them P1 CONN_01X06, SW1 SW_Push, U1 BP, U2 RFM69, U3 M24M02-DR

Commit message: Ready for ordering
Parts:
- AE1: footprint BP:U.FL-COAX -> RFM69:U.FL-COAX
Changed lines of the file:
@@
 LIBS:mechanical
 LIBS:m24m02-dr
-LIBS:BP-Extension-cache
+LIBS:BPnode-BB-cache
 EELAYER 25 0
 EELAYER END
@@
 F 0 "AE1" H 9425 4875 50  0000 R CNN
 F 1 "Antenna_Shield" H 9425 4800 50  0000 R CNN
-F 2 "BP:U.FL-COAX" H 9500 4800 50  0001 C CNN
+F 2 "RFM69:U.FL-COAX" H 9500 4800 50  0001 C CNN
 F 3 "" H 9500 4800 50  0001 C CNN
 	1    9500 4700
