File: KiCAD/BPnode-BB.kicad_pcb (KiCad board)
At the start: 2 copper layers, 19.8 x 49.3 mm, 10 parts, among them P1 CONN_01X06, SW1 SW_Push, U1 BP, U2 RFM69, U3 M24M02-DR

Commit message: Ready for ordering
Parts:
- AE1: footprint BP:U.FL-COAX -> RFM69:U.FL-COAX
Routing:
- net GND: track 77.9 -> 78.9 mm
- net MOSI: track 23.6 -> 24.4 mm
- net DIO0: track 5.92 -> 6.65 mm
- net SSEL: track 6.26 -> 6.82 mm
- net DIO1: track 11.6 -> 11.1 mm
- net SCLK: track 10.6 -> 11.1 mm
- net Net-(AE1-Pad1): track 6.30 -> 5.80 mm
- net DIO3: track 13.7 -> 13.2 mm
- net DIO2: track 18.5 -> 19.0 mm
Other:
- outline, holes or cut-outs redrawn
- board text added: "B6"
- board text added: "B7"
- board text added: "Reset Button"
- board text added: "https://github.com/tht/bpnode-bb"

Commit message: Ready for ordering
Routing:
- net +3V3: track 74.0 -> 72.0 mm
- net Vin: track 57.3 -> 56.7 mm

Commit message: Rev 2 as ordered
Other:
- board text added: "Rev 2 2017/03"
- board text removed: "Rev 2 2017/02"
Changed lines of the file:
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@@
     (links 42)
     (no_connects 0)
-    (area 138.608999 79.172999 158.571001 128.599001)
+    (area 137.147 70.567999 158.877001 131.939)
     (thickness 1.6)
     (drawings 63)
@@
     (effects (font (size 0.8 0.8) (thickness 0.15)))
   )
-  (gr_text "Rev 2\n2017/02" (at 148.463 118.872) (layer F.SilkS)
+  (gr_text "Rev 2\n2017/03" (at 148.463 118.872) (layer F.SilkS)
     (effects (font (size 0.8 0.8) (thickness 0.15)) (justify left))
   )
